Commit message: fixed model issues

File: src/nav-sim/urdf/xacro/base.xacro (robot description, xacro)
@@ -78,5 +78,5 @@
         <xacro:cylinder_inertial_matrix m="${wheel_m}" r="${wheel_radius}" h="${wheel_length}" />
       </link>
-      <joint name="${name}_wheel2base_link" type="continuous">
+      <joint name="base_${name}_wheel_joint" type="continuous">
         <parent link="base_link" />
         <child link="${name}_wheel" />
@@ -88,6 +88,6 @@
       </gazebo>
     </xacro:macro>
-    <xacro:add_wheels name="left" flag="1" />
-    <xacro:add_wheels name="right" flag="-1" />
+    <xacro:add_wheels name="l" flag="1" />
+    <xacro:add_wheels name="r" flag="-1" />
     <!-- 支撑轮 -->
     <!-- 支撑轮属性 -->

File: src/nav-sim/urdf/xacro/car_gazebo.xacro (robot description, xacro)
@@ -12,56 +12,3 @@
     <!-- kinect仿真的 xacro 文件 -->
     <xacro:include filename="sensors_kinect.xacro" />
-  <!-- Transmission is important to link the joints and the controller -->
-  <transmission name="left_wheel_joint_trans">
-    <type>transmission_interface/SimpleTransmission</type>
-    <joint name="left_wheel_joint">
-      <hardwareInterface>hardware_interface/VelocityJointInterface</hardwareInterface>
-    </joint>
-    <actuator name="left_wheel_joint_motor">
-      <hardwareInterface>hardware_interface/VelocityJointInterface</hardwareInterface>
-      <mechanicalReduction>1</mechanicalReduction>
-    </actuator>
-  </transmission>
-  <!-- Transmission is important to link the joints and the controller -->
-  <transmission name="right_wheel_joint_trans">
-    <type>transmission_interface/SimpleTransmission</type>
-    <joint name="right_wheel_joint">
-      <hardwareInterface>hardware_interface/VelocityJointInterface</hardwareInterface>
-    </joint>
-    <actuator name="right_wheel_joint_motor">
-      <hardwareInterface>hardware_interface/VelocityJointInterface</hardwareInterface>
-      <mechanicalReduction>1</mechanicalReduction>
-    </actuator>
-  </transmission>
-  <gazebo>
-    <plugin filename="libgazebo_ros_diff_drive.so" name="differential_drive_controller">
-      <rosDebugLevel>Debug</rosDebugLevel>
-      <publishWheelTF>true</publishWheelTF>
-      <robotNamespace>/</robotNamespace>
-      <publishTf>1</publishTf>
-      <publishWheelJointState>true</publishWheelJointState>
-      <alwaysOn>true</alwaysOn>
-      <updateRate>100.0</updateRate>
-      <legacyMode>true</legacyMode>
-      <leftJoint>left_wheel_joint</leftJoint>
-      <!--left_joint-->
-      <rightJoint>right_wheel_joint</rightJoint>
-      <!--right_joint-->
-      <wheelSeparation>0.277</wheelSeparation>
-      <!--wheel_separation-->
-      <wheelDiameter>0.073</wheelDiameter>
-      <!--wheel_diameter-->
-      <broadcastTF>1</broadcastTF>
-      <wheelTorque>30</wheelTorque>
-      <wheelAcceleration>1.8</wheelAcceleration>
-      <commandTopic>cmd_vel</commandTopic>
-      <odometryFrame>odom</odometryFrame>
-      <odometryTopic>odom</odometryTopic>
-      <robotBaseFrame>base_footprint</robotBaseFrame>
-      <!--
-            <odometrySource>world</odometrySource>
-            <publishTf>1</publishTf>
-            -->
-    </plugin>
-  </gazebo>
 </robot>

File: src/nav-sim/urdf/xacro/move.xacro (robot description, xacro)
@@ -15,19 +15,19 @@
     </xacro:macro>
     <!-- 每一个驱动轮都需要配置传动装置 -->
-    <xacro:joint_trans joint_name="left_wheel2base_link" />
-    <xacro:joint_trans joint_name="right_wheel2base_link" />
+    <xacro:joint_trans joint_name="base_l_wheel_joint" />
+    <xacro:joint_trans joint_name="base_r_wheel_joint" />
     <!-- 控制器 -->
     <gazebo>
         <plugin name="differential_drive_controller" filename="libgazebo_ros_diff_drive.so">
             <rosDebugLevel>Debug</rosDebugLevel>
-            <publishWheelTF>true</publishWheelTF>
+            <publishWheelTF>false</publishWheelTF>
             <robotNamespace>/</robotNamespace>
             <publishTf>1</publishTf>
-            <publishWheelJointState>true</publishWheelJointState>
+            <publishWheelJointState>false</publishWheelJointState>
             <alwaysOn>true</alwaysOn>
             <updateRate>100.0</updateRate>
             <legacyMode>true</legacyMode>
-            <leftJoint>left_wheel2base_link</leftJoint> <!-- 左轮 -->
-            <rightJoint>right_wheel2base_link</rightJoint> <!-- 右轮 -->
+            <leftJoint>base_l_wheel_joint</leftJoint> <!-- 左轮 -->
+            <rightJoint>base_r_wheel_joint</rightJoint> <!-- 右轮 -->
             <wheelSeparation>${base_link_radius * 2}</wheelSeparation> <!-- 车轮间距 -->
             <wheelDiameter>${wheel_radius * 2}</wheelDiameter> <!-- 车轮直径 -->
@@ -36,4 +36,5 @@
             <wheelAcceleration>1.8</wheelAcceleration>
             <commandTopic>cmd_vel</commandTopic> <!-- 运动控制话题 -->
+            <publishOdomTF>false</publishOdomTF>
             <odometryFrame>odom</odometryFrame>
             <odometryTopic>odom</odometryTopic> <!-- 里程计话题 -->
