Commit message: fixed model issues

File: src/gz_sim/urdf/xacro/car_gazebo.xacro (robot description, xacro)
@@ -12,56 +12,3 @@
     <!-- kinect仿真的 xacro 文件 -->
     <xacro:include filename="sensors_kinect.xacro" />
-      <!-- Transmission is important to link the joints and the controller -->
-  <transmission name="left_wheel_joint_trans">
-    <type>transmission_interface/SimpleTransmission</type>
-    <joint name="left_wheel_joint">
-      <hardwareInterface>hardware_interface/VelocityJointInterface</hardwareInterface>
-    </joint>
-    <actuator name="left_wheel_joint_motor">
-      <hardwareInterface>hardware_interface/VelocityJointInterface</hardwareInterface>
-      <mechanicalReduction>1</mechanicalReduction>
-    </actuator>
-  </transmission>
-  <!-- Transmission is important to link the joints and the controller -->
-  <transmission name="right_wheel_joint_trans">
-    <type>transmission_interface/SimpleTransmission</type>
-    <joint name="right_wheel_joint">
-      <hardwareInterface>hardware_interface/VelocityJointInterface</hardwareInterface>
-    </joint>
-    <actuator name="right_wheel_joint_motor">
-      <hardwareInterface>hardware_interface/VelocityJointInterface</hardwareInterface>
-      <mechanicalReduction>1</mechanicalReduction>
-    </actuator>
-  </transmission>
-  <gazebo>
-    <plugin filename="libgazebo_ros_diff_drive.so" name="differential_drive_controller">
-      <rosDebugLevel>Debug</rosDebugLevel>
-      <publishWheelTF>true</publishWheelTF>
-      <robotNamespace>/</robotNamespace>
-      <publishTf>1</publishTf>
-      <publishWheelJointState>true</publishWheelJointState>
-      <alwaysOn>true</alwaysOn>
-      <updateRate>100.0</updateRate>
-      <legacyMode>true</legacyMode>
-      <leftJoint>left_wheel_joint</leftJoint>
-      <!--left_joint-->
-      <rightJoint>right_wheel_joint</rightJoint>
-      <!--right_joint-->
-      <wheelSeparation>0.277</wheelSeparation>
-      <!--wheel_separation-->
-      <wheelDiameter>0.073</wheelDiameter>
-      <!--wheel_diameter-->
-      <broadcastTF>1</broadcastTF>
-      <wheelTorque>30</wheelTorque>
-      <wheelAcceleration>1.8</wheelAcceleration>
-      <commandTopic>cmd_vel</commandTopic>
-      <odometryFrame>odom</odometryFrame>
-      <odometryTopic>odom</odometryTopic>
-      <robotBaseFrame>base_footprint</robotBaseFrame>
-      <!--
-            <odometrySource>world</odometrySource>
-            <publishTf>1</publishTf>
-            -->
-    </plugin>
-  </gazebo>
 </robot>
